Commit message: try drawer collision activation

File: panda_gym/assets/drawer/drawer_with_handle.urdf (robot description, URDF)
Before this commit: robot drawer_with_handle, 3 links, 2 joints
Joints:
- joint handle_fixed: origin xyz=0 -0.18 0 rpy=0 0 0 -> xyz=0 -0.28 0 rpy=0 0 0

Commit message: changed some parameters and limits

File: panda_gym/assets/drawer/drawer_with_handle.urdf (robot description, URDF)
Before this commit: robot drawer_with_handle, 3 links, 2 joints
Joints:
- joint drawer_slide: limit lower=0 upper=0.15 effort=10.0 velocity=1.0 -> lower=0.4 upper=0.4 effort=1.0 velocity=1.0

Commit message: changed limits

File: panda_gym/assets/drawer/drawer_with_handle.urdf (robot description, URDF)
Before this commit: robot drawer_with_handle, 3 links, 2 joints
Joints:
- joint drawer_slide: limit lower=0.4 upper=0.4 effort=1.0 velocity=1.0 -> lower=-0.8 upper=0.8 effort=1.0 velocity=1.0

Commit message: placed drawer slightly outside of box

File: panda_gym/assets/drawer/drawer_with_handle.urdf (robot description, URDF)
Before this commit: robot drawer_with_handle, 3 links, 2 joints
Joints:
- joint drawer_slide: origin xyz=0 0 0.05 rpy=0 0 0 -> xyz=0 0.1 0.05 rpy=0 0 0

Commit message: changed direction of placement

File: panda_gym/assets/drawer/drawer_with_handle.urdf (robot description, URDF)
Before this commit: robot drawer_with_handle, 3 links, 2 joints
Joints:
- joint drawer_slide: origin xyz=0 0.1 0.05 rpy=0 0 0 -> xyz=0 -0.1 0.05 rpy=0 0 0

Commit message: changed handle placement back and friction coefficients

File: panda_gym/assets/drawer/drawer_with_handle.urdf (robot description, URDF)
Before this commit: robot drawer_with_handle, 3 links, 2 joints
Joints:
- joint handle_fixed: origin xyz=0 -0.28 0 rpy=0 0 0 -> xyz=0 -0.18 0 rpy=0 0 0

Commit message: changed limits

File: panda_gym/assets/drawer/drawer_with_handle.urdf (robot description, URDF)
Before this commit: robot drawer_with_handle, 3 links, 2 joints
Joints:
- joint drawer_slide: limit lower=-0.8 upper=0.8 effort=1.0 velocity=1.0 -> lower=-0.4 upper=0.4 effort=1.0 velocity=1.0

Commit message: changed design of drawer

File: panda_gym/assets/drawer/drawer_with_handle.urdf (robot description, URDF)
Before this commit: robot drawer_with_handle, 3 links, 2 joints
Links:
- link handle: geometry collision cylinder length=0.06 radius=0.02; visual cylinder length=0.06 radius=0.02
Joints:
- joint drawer_slide: axis 0 1 0 -> 0 -1 0; origin xyz=0 -0.1 0.05 rpy=0 0 0 -> xyz=0 -0.055 0.03 rpy=0 0 0
